File: PCBs/Lab4/Lab4.kicad_sch (KiCad schematic)
At the start: 13 parts, among them IC1 M0C1103QDDFRQ1, J1 Conn_01x05_Pin, SW1 SW_SPST, SW2 SW_SPST

Commit message: Complete Labs 1-6: firmware and PCB submissions
Labs 1-3: GPIO/state machine LED control with button input
Lab 4: KiCad Simon PCB design
Lab 5: PWM buzzer + Mary Had a Little Lamb state machine
Lab 6: SPI RGB LED control synchronized to song and button presses
Parts:
- removed D3: NeoPixel_THT, LED_THT:LED_D5.0mm-4_RGB_Staggered_Pins, symbol LED:NeoPixel_THT
- removed SW2: SW_SPST, Button_Switch_SMD:SW_SPST_PTS647_Sx50, symbol Switch:SW_SPST
Other:
- moved on the sheet: D2
